File: vejas-pi/vejas-pi.kicad_pcb (KiCad board)
At the start: 2 copper layers, 21 x 51 mm, 33 parts, among them J1 USB_C_Receptacle_USB2.0_14P, J2 Conn_01x20_Pin, J3 Conn_01x20_Pin, J4 Conn_01x03_Pin, SW1 SW_Push, U1 RP2040, U3 W25Q128JVS, U4 MCP1700x-330xxTT, Y1 12MHz

Commit message: a lot of pcb
Parts:
- moved C4 47.1 mm to (124.4, 57.7)
- moved C9 46.8 mm to (119.8, 63.0), turned to -90 degrees
- moved C12 43.5 mm to (120.8, 63.4), turned to -90 degrees
- moved C3 41.1 mm to (123.6, 45.8), turned to 90 degrees
- moved C8 41.1 mm to (112.6, 59.3), turned to -90 degrees
- moved C1 40.6 mm to (122.9, 42.3)
- moved C2 40.2 mm to (122.9, 43.3)
- moved R1 39.7 mm to (121.4, 37.0), turned to -90 degrees
- moved R4 38.6 mm to (120.8, 41.1), turned to -90 degrees
- moved C5 38.4 mm to (122.5, 45.8), turned to 90 degrees
- moved C11 38.3 mm to (122.4, 51.2), turned to 45 degrees
- moved R3 38.1 mm to (119.6, 41.1), turned to -90 degrees
- moved C7 37.7 mm to (114.0, 52.0), turned to 135 degrees
- moved C10 37.1 mm to (120.7, 49.7), turned to 90 degrees
- moved C6 36.6 mm to (121.3, 45.8), turned to 90 degrees
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Routing:
- net +3V3: track 0.00 -> 57.3 mm, vias 0 -> 4
- net GPIO0: track 0.00 -> 28.3 mm
- net GPIO1: track 0.00 -> 25.9 mm
- net GPIO29_ADC3: track 0.00 -> 25.8 mm
- net SWD: track 0.00 -> 24.9 mm, vias 0 -> 1
- net GPIO16: track 0.00 -> 22.3 mm
- net GPIO28_ADC2: track 0.00 -> 22.1 mm
- net GPIO2: track 0.00 -> 22.0 mm
- net GPIO15: track 0.00 -> 20.3 mm
- net SWCLK: track 0.00 -> 19.6 mm
- net GPIO17: track 0.00 -> 19.0 mm
- net GPIO14: track 0.00 -> 17.6 mm
- net GPIO27_ADC1: track 0.00 -> 17.6 mm
- net GND: track 0.00 -> 17.3 mm, vias 0 -> 13
- net RUN: track 0.00 -> 17.0 mm, vias 0 -> 1
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- added copper zone on B.Cu, net GND
- added copper zone on F.Cu, net GND

Commit message: pcb
Parts:
- J2, J3, J4: moved to B.Cu
- moved J4 5.12 mm to (121.3, 76.7)
- moved C5 3.75 mm to (121.9, 49.5)
- moved C6 3.75 mm to (120.8, 49.5)
- moved C10 2.37 mm to (119.4, 47.7)
- moved U3 1.36 mm to (116.6, 48.7)
- moved C17 1.35 mm to (116.9, 46.7)
- moved C11 1.22 mm to (123.5, 51.6)
- moved R6 0.82 mm to (114.0, 47.2)
- moved SW1 0.71 mm to (116.0, 44.4)
- moved R7 0.51 mm to (119.3, 45.5)
- moved C7 0.40 mm to (114.4, 51.8)
- turned J2 to 180 degrees
- turned J3 to 180 degrees
Routing:
- net GPIO4: track 0.00 -> 15.7 mm
- net GPIO3: track 5.41 -> 20.2 mm
- net SWD: track 24.9 -> 20.5 mm, vias 1 -> 0
- net Net-(U1-USB_DP): track 12.8 -> 17.1 mm
- net Net-(U1-USB_DM): track 12.8 -> 17.0 mm
- net +3V3: track 57.3 -> 60.9 mm, vias 4 -> 2
- net SWCLK: track 19.6 -> 23.0 mm
- net +1V1: track 10.1 -> 13.4 mm
- net GND: track 17.3 -> 19.3 mm, vias 13 -> 11
- net QSPI_SS: track 14.3 -> 12.7 mm
- net QSPI_SD02: track 3.53 -> 5.00 mm
- net GPIO5: track 15.7 -> 17.2 mm
- net GPIO6: track 11.4 -> 12.6 mm
- net QSPI_SD0: track 3.25 -> 3.80 mm
- net QSPI_SD3: track 5.60 -> 5.74 mm, vias 2 -> 0

Commit message: pcb
Parts:
- added D2: WS2812B-2020, LED_SMD:LED_WS2812B-2020_PLCC4_2.0x2.0mm, F.Cu at (123.6, 38.7)
- added D3: 1N4148, Diode_SMD:D_SOD-323, F.Cu at (123.7, 36.3)
- moved C3 7.27 mm to (123.5, 53.1)
- moved C11 0.48 mm to (123.7, 51.2)
Connections:
- U1 pad 37: unconnected-(U1-GPIO25-Pad37) -> LED
Routing:
- net +3V3: track 60.9 -> 80.3 mm, vias 2 -> 6
- net LED: track 0.00 -> 19.1 mm, vias 0 -> 2
- net GND: track 19.3 -> 36.0 mm, vias 11 -> 17
- net VBUS: track 11.3 -> 25.2 mm, vias 0 -> 2
- net +1V1: track 13.4 -> 26.4 mm, vias 0 -> 3
- net Net-(D2-VSS): track 0.00 -> 4.06 mm
- net GPIO4: track 15.7 -> 17.7 mm, vias 0 -> 1
- net GPIO29_ADC3: track 25.8 -> 26.3 mm

Commit message: pcb v1
Parts:
- added G***: LOGO, LOGO, F.Cu at (118.7, 74.3)
- added R8: 1K, Resistor_SMD:R_0402_1005Metric, F.Cu at (122.0, 68.1)
- added SW2: SW_Push, Button_Switch_SMD:SW_Push_SPST_NO_Alps_SKRK, F.Cu at (118.7, 71.4)
Routing:
- net RUN: track 17.0 -> 22.4 mm, vias 1 -> 2
- net Net-(R8-Pad1): track 0.00 -> 3.26 mm
- net GND: track 36.0 -> 35.1 mm, vias 17 -> 19
- net +3V3: track 80.3 -> 79.5 mm
- net XOUT: track 4.54 -> 3.85 mm
Other:
- board text added: "VejasRP2040"
- board text added: "lasvejas"

Commit message: pcb
Parts:
- moved G*** 6.70 mm to (113.5, 70.0), turned to 90 degrees

Commit message: very kul
Parts:
- removed J4: Conn_01x03_Pin, Connector_PinHeader_2.54mm:PinHeader_1x03_P2.54mm_Vertical
- added J5: MSD-12-A, MSD-12-A:CUI_MSD-12-A, B.Cu at (118.7, 67.4)
- R3, R4: value 27 -> 27.4
Routing:
- net SWCLK: track 23.0 -> 14.5 mm
- net SWD: track 20.5 -> 15.6 mm
- net RUN: track 22.4 -> 23.2 mm

Commit message: cool stuff V1.1 SHIPPED
Parts:
- removed D3: 1N4148, Diode_SMD:D_SOD-323
- removed J5: MSD-12-A, MSD-12-A:CUI_MSD-12-A
- added C18: 0.1uF, Capacitor_SMD:C_0402_1005Metric, F.Cu at (121.8, 73.8)
- added U2: LIS3DH, Package_LGA:LGA-16_3x3mm_P0.5mm_LayoutBorder3x5y, F.Cu at (118.7, 75.6)
- J1: footprint Connector_USB:USB_C_Receptacle_HRO_TYPE-C-31-M-12 -> Connector_USB:USB_C_Receptacle_JAE_DX07S016JA1R1500
- moved R8 0.28 mm to (121.7, 68.1)
- moved J1 0.27 mm to (118.8, 30.2)
Connections:
- D2 pad 2: Net-(D2-VSS) -> GND
- D2 pad 4: GND -> VBUS
- J2 pad 16: GPIO19 -> unconnected-(J2-Pin_16-Pad16)
- J2 pad 17: GPIO18 -> unconnected-(J2-Pin_17-Pad17)
- J2 pad 19: GPIO17 -> SWD
- J2 pad 20: GPIO16 -> SWCLK
Routing:
- net GND: track 35.1 -> 62.7 mm, vias 19 -> 24
- net +3V3: track 79.5 -> 104.6 mm, vias 6 -> 8
- net GPIO19: track 11.7 -> 27.2 mm, vias 0 -> 2
- net GPIO18: track 12.8 -> 24.5 mm, vias 0 -> 2
- net SWCLK: track 14.5 -> 23.3 mm, vias 0 -> 1
- net GPIO17: track 19.0 -> 25.9 mm, vias 0 -> 2
- net Net-(D2-VSS): track 4.06 -> 0.00 mm
- net SWD: track 15.6 -> 19.6 mm, vias 0 -> 1
- net VBUS: track 25.2 -> 28.8 mm, vias 2 -> 4
- net GPIO16: track 22.3 -> 25.3 mm
- net USB_D-: track 10.1 -> 10.9 mm
- net Net-(J1-CC2): track 2.71 -> 3.38 mm
- net USB_D+: track 9.45 -> 8.83 mm
- net Net-(J1-CC1): track 3.11 -> 3.62 mm
