File: vejas-pi/vejas-pi.kicad_sch (KiCad schematic)
At the start: 33 parts, among them J1 USB_C_Receptacle_USB2.0_14P, J2 Conn_01x20_Pin, J3 Conn_01x20_Pin, J4 Conn_01x03_Pin, SW1 SW_Push, U1 RP2040, U3 W25Q128JVS, U4 MCP1700x-330xxTT, Y1 12MHz

Commit message: a lot of pcb
Changed lines of the file:
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@@
 	)
 	(junction
+		(at 60.96 152.4)
+		(diameter 0)
+		(color 0 0 0 0)
+	)
+	(junction
 		(at 210.82 22.86)
 		(diameter 0)
@@
 	(wire
 		(pts
+			(xy 60.96 149.86) (xy 60.96 152.4)
+		)
+		(stroke
+			(width 0)
+			(type default)
+		)
+	)
+	(wire
+		(pts
 			(xy 170.18 86.36) (xy 168.91 86.36)
 		)
@@
 	(wire
 		(pts
-			(xy 52.07 152.4) (xy 63.5 152.4)
+			(xy 52.07 152.4) (xy 60.96 152.4)
 		)
 		(stroke
@@
 	(wire
 		(pts
+			(xy 60.96 152.4) (xy 63.5 152.4)
+		)
+		(stroke
+			(width 0)
+			(type default)
+		)
+	)
+	(wire
+		(pts
 			(xy 57.15 11.43) (xy 58.42 11.43)
 		)
@@
 	(global_label "QSPI_SS"
 		(shape input)
-		(at 60.96 152.4 90)
+		(at 60.96 149.86 90)
 		(fields_autoplaced yes)
 		(effects
@@
 		)
 		(property "Intersheetrefs" "${INTERSHEET_REFS}"
-			(at 60.96 141.6134 90)
+			(at 60.96 139.0734 90)
 			(effects
 				(font

Commit message: pcb
Parts:
- added D2: WS2812B-2020, LED_SMD:LED_WS2812B-2020_PLCC4_2.0x2.0mm, symbol LED:WS2812B-2020
- added D3: 1N4148, Diode_SMD:D_SOD-323, symbol Device:D
Connections:
- net GND: now also D2.4 (VDD)
- net VBUS: now also D3.2 (A)
- net LED: now reaches U1.37 (GPIO25)
- net LED: now also D2.3 (DIN)
- new net: D2.2 (VSS), D3.1 (K)
- no-connect marks 1 -> 0

Commit message: pcb v1
Parts:
- added R8: 1K, Resistor_SMD:R_0402_1005Metric, symbol Device:R
- added SW2: SW_Push, Button_Switch_SMD:SW_Push_SPST_NO_Alps_SKRK, symbol Switch:SW_Push
Connections:
- net GND: now also SW2.1
- net RUN: now also R8.2
- new net: R8.1, SW2.2

Commit message: very kul
Parts:
- removed J4: Conn_01x03_Pin, Connector_PinHeader_2.54mm:PinHeader_1x03_P2.54mm_Vertical, symbol Connector:Conn_01x03_Pin
- added J5: MSD-12-A, MSD-12-A:CUI_MSD-12-A, symbol MSD-12-A:MSD-12-A
- R3, R4: value 27 -> 27.4
Connections:
- net +3V3: now also J5.P4 (VDD)
- net GND: now also J5.G1 (COVER_GND), J5.G2 (COVER_GND__1), J5.G3 (COVER_GND__2), J5.G4 (COVER_GND__3), J5.G5 (COVER_GND__4), J5.G6 (COVER_GND__5), J5.P6 (VSS)
Other:
- moved on the sheet: C1, C10, C11, C12, C2, C3, C4, C5, C6, C7, C8, C9

Commit message: cool stuff V1.1 SHIPPED
Parts:
- removed D3: 1N4148, Diode_SMD:D_SOD-323, symbol Device:D
- removed J5: MSD-12-A, MSD-12-A:CUI_MSD-12-A, symbol MSD-12-A:MSD-12-A
- added C18: 0.1uF, Capacitor_SMD:C_0402_1005Metric, symbol Device:C
- added U2: LIS3DH, Package_LGA:LGA-16_3x3mm_P0.5mm_LayoutBorder3x5y, symbol Sensor_Motion:LIS3DH
- J1: footprint Connector_USB:USB_C_Receptacle_HRO_TYPE-C-31-M-12 -> Connector_USB:USB_C_Receptacle_JAE_DX07S016JA1R1500
Connections:
- net +3V3: now also C18.1, U2.1 (VDD_IO), U2.14 (VDD)
- net GND: now also D2.2 (VSS), C18.2, U2.10 (GND), U2.12 (GND), U2.5 (GND); no longer D2.4 (VDD)
- net GPIO16: now also U2.7 (SDO); no longer J2.20 (Pin_20)
- net GPIO17: now also U2.8 (CS); no longer J2.19 (Pin_19)
- net GPIO18: now also U2.4 (SPC); no longer J2.17 (Pin_17)
- net GPIO19: now also U2.6 (SDI); no longer J2.16 (Pin_16)
- net SWCLK: now also J2.20 (Pin_20)
- net SWD: now also J2.19 (Pin_19)
- net VBUS: now also D2.4 (VDD)
- no-connect marks 0 -> 7
Other:
- moved on the sheet: D2
